File: Hardware/GVH_InteractiveCounter/GVH_InteractiveCounter.kicad_pcb (KiCad board)
At the start: 2 copper layers, 0 parts

Commit message: Saving before changing from 1206 to 0805 components
Parts:
- added C1: 0.1uF, Capacitor_SMD:C_1206_3216Metric_Pad1.33x1.80mm_HandSolder, F.Cu at (63.5, 95.1)
- added C2: 22nF, Capacitor_SMD:C_1206_3216Metric_Pad1.33x1.80mm_HandSolder, F.Cu at (73.4, 94.3)
- added D1: Touch_Indicator, LED_SMD:LED_1206_3216Metric_Pad1.42x1.75mm_HandSolder, F.Cu at (59.7, 95.1)
- added J1: Molex Micro-Fit, 0_connector:MOLEX_MICROFIT-RA-5POS_436500500, F.Cu at (88.6, 47.8)
- added J2: Molex Micro-Fit, 0_connector:MOLEX_MICROFIT-RA-5POS_436500500, F.Cu at (136.0, 58.0)
- added J3: Molex Ultra-Fit, 0_connector:MOLEX_ULTRAFIT-RA-2POS_1723104102, F.Cu at (204.6, 80.4)
- added J4: Electrode, Connector_Pin:Pin_D1.3mm_L11.0mm_LooseFit, F.Cu at (85.0, 91.7)
- added JP1: SolderJumper_2_Bridged, Jumper:SolderJumper-2_P1.3mm_Bridged_RoundedPad1.0x1.5mm, F.Cu at (68.2, 96.8)
- added JP10: SolderJumper_3_Bridged12, Jumper:SolderJumper-3_P1.3mm_Bridged12_RoundedPad1.0x1.5mm, F.Cu at (205.5, 116.6)
- added JP9: SolderJumper_3_Bridged12, Jumper:SolderJumper-3_P1.3mm_Bridged12_RoundedPad1.0x1.5mm, F.Cu at (204.8, 123.6)
- added R1: 1K, Resistor_SMD:R_1206_3216Metric_Pad1.30x1.75mm_HandSolder, F.Cu at (55.9, 95.1)
- added R2: 10K, Resistor_SMD:R_1206_3216Metric_Pad1.30x1.75mm_HandSolder, F.Cu at (79.1, 91.7)
- added U1: AT42QT1010, 0_sensor:AT42QT1010-TSGR_1, F.Cu at (67.7, 93.5)
- added U8: SN74HC165DR, Package_SO:SOIC-16W_5.3x10.2mm_P1.27mm, F.Cu at (187.7, 104.8)
- added U9: 74HCT2G34GW_125, 0_integrated_circuits:74HCT2G34GW_125_SOT363, F.Cu at (223.9, 121.8)
Routing:
- net Net-(U1-SNSK): track 0.00 -> 14.8 mm
- net Net-(U1-SNS): track 0.00 -> 9.67 mm
- net Net-(D1-A): track 0.00 -> 9.05 mm
- net Net-(J4-Pin_1): track 0.00 -> 4.29 mm
- net VCC: track 0.00 -> 4.04 mm
- net Net-(D1-K): track 0.00 -> 3.84 mm
- net /Touch Sensor 1/TOUCH SENSE: track 0.00 -> 2.36 mm
Other:
- board outline added: 355.6 x 25.4 mm

Commit message: Backing up work on PCB before some major changes
Parts:
- added C10: 22nF, Capacitor_SMD:C_0805_2012Metric_Pad1.18x1.45mm_HandSolder, F.Cu at (228.8, 92.0)
- added C11: 0.1uF, Capacitor_SMD:C_0805_2012Metric_Pad1.18x1.45mm_HandSolder, F.Cu at (262.1, 92.2)
- added C12: 22nF, Capacitor_SMD:C_0805_2012Metric_Pad1.18x1.45mm_HandSolder, F.Cu at (271.9, 92.0)
- added C13: 0.1uF, Capacitor_SMD:C_0805_2012Metric_Pad1.18x1.45mm_HandSolder, F.Cu at (304.0, 92.2)
- added C14: 22nF, Capacitor_SMD:C_0805_2012Metric_Pad1.18x1.45mm_HandSolder, F.Cu at (313.8, 92.0)
- added C15: 0.1uF, Capacitor_SMD:C_0805_2012Metric_Pad1.18x1.45mm_HandSolder, F.Cu at (345.9, 92.2)
- added C16: 22nF, Capacitor_SMD:C_0805_2012Metric_Pad1.18x1.45mm_HandSolder, F.Cu at (355.8, 92.0)
- added C17: 0.1uF, Capacitor_SMD:C_0805_2012Metric_Pad1.18x1.45mm_HandSolder, F.Cu at (115.0, 58.7)
- added C18: 0.1uF, Capacitor_SMD:C_0805_2012Metric_Pad1.18x1.45mm_HandSolder, F.Cu at (115.0, 61.7)
- added C3: 0.1uF, Capacitor_SMD:C_0805_2012Metric_Pad1.18x1.45mm_HandSolder, F.Cu at (100.0, 91.5)
- added C4: 22nF, Capacitor_SMD:C_0805_2012Metric_Pad1.18x1.45mm_HandSolder, F.Cu at (109.8, 91.3)
- added C5: 0.1uF, Capacitor_SMD:C_0805_2012Metric_Pad1.18x1.45mm_HandSolder, F.Cu at (135.4, 91.5)
- added C6: 22nF, Capacitor_SMD:C_0805_2012Metric_Pad1.18x1.45mm_HandSolder, F.Cu at (145.2, 91.3)
- added C7: 0.1uF, Capacitor_SMD:C_0805_2012Metric_Pad1.18x1.45mm_HandSolder, F.Cu at (175.8, 92.2)
- added C8: 22nF, Capacitor_SMD:C_0805_2012Metric_Pad1.18x1.45mm_HandSolder, F.Cu at (185.6, 92.0)
- added C9: 0.1uF, Capacitor_SMD:C_0805_2012Metric_Pad1.18x1.45mm_HandSolder, F.Cu at (218.9, 92.2)
- added D2: Touch_Indicator, LED_SMD:LED_0805_2012Metric_Pad1.15x1.40mm_HandSolder, F.Cu at (96.6, 92.4)
- added D3: Touch_Indicator, LED_SMD:LED_0805_2012Metric_Pad1.15x1.40mm_HandSolder, F.Cu at (132.0, 92.4)
- added D4: Touch_Indicator, LED_SMD:LED_0805_2012Metric_Pad1.15x1.40mm_HandSolder, F.Cu at (172.3, 93.1)
- added D5: Touch_Indicator, LED_SMD:LED_0805_2012Metric_Pad1.15x1.40mm_HandSolder, F.Cu at (215.5, 93.1)
- added D6: Touch_Indicator, LED_SMD:LED_0805_2012Metric_Pad1.15x1.40mm_HandSolder, F.Cu at (258.7, 93.1)
- added D7: Touch_Indicator, LED_SMD:LED_0805_2012Metric_Pad1.15x1.40mm_HandSolder, F.Cu at (300.6, 93.1)
- added D8: Touch_Indicator, LED_SMD:LED_0805_2012Metric_Pad1.15x1.40mm_HandSolder, F.Cu at (342.5, 93.1)
- added J10: Electrode, Connector_Pin:Pin_D1.3mm_L11.0mm_LooseFit, F.Cu at (321.8, 91.9)
- added J11: Electrode, Connector_Pin:Pin_D1.3mm_L11.0mm_LooseFit, F.Cu at (363.7, 91.9)
- added J5: Electrode, Connector_Pin:Pin_D1.3mm_L11.0mm_LooseFit, F.Cu at (117.8, 91.3)
- added J6: Electrode, Connector_Pin:Pin_D1.3mm_L11.0mm_LooseFit, F.Cu at (153.2, 91.2)
- added J7: Electrode, Connector_Pin:Pin_D1.3mm_L11.0mm_LooseFit, F.Cu at (193.5, 91.9)
- added J8: Electrode, Connector_Pin:Pin_D1.3mm_L11.0mm_LooseFit, F.Cu at (236.7, 91.9)
- added J9: Electrode, Connector_Pin:Pin_D1.3mm_L11.0mm_LooseFit, F.Cu at (279.9, 91.9)
- added JP2: SolderJumper_2_Bridged, Jumper:SolderJumper-2_P1.3mm_Bridged_RoundedPad1.0x1.5mm, F.Cu at (96.5, 90.1)
- added JP3: SolderJumper_2_Bridged, Jumper:SolderJumper-2_P1.3mm_Bridged_RoundedPad1.0x1.5mm, F.Cu at (131.9, 90.1)
- added JP4: SolderJumper_2_Bridged, Jumper:SolderJumper-2_P1.3mm_Bridged_RoundedPad1.0x1.5mm, F.Cu at (172.3, 90.8)
- added JP5: SolderJumper_2_Bridged, Jumper:SolderJumper-2_P1.3mm_Bridged_RoundedPad1.0x1.5mm, F.Cu at (215.5, 90.8)
- added JP6: SolderJumper_2_Bridged, Jumper:SolderJumper-2_P1.3mm_Bridged_RoundedPad1.0x1.5mm, F.Cu at (258.7, 90.8)
- added JP7: SolderJumper_2_Bridged, Jumper:SolderJumper-2_P1.3mm_Bridged_RoundedPad1.0x1.5mm, F.Cu at (300.6, 90.8)
- added JP8: SolderJumper_2_Bridged, Jumper:SolderJumper-2_P1.3mm_Bridged_RoundedPad1.0x1.5mm, F.Cu at (342.5, 90.8)
- added R10: 10K, Resistor_SMD:R_0805_2012Metric_Pad1.20x1.40mm_HandSolder, F.Cu at (231.7, 92.0)
- added R11: 1K, Resistor_SMD:R_0805_2012Metric_Pad1.20x1.40mm_HandSolder, F.Cu at (255.2, 92.1)
- added R12: 10K, Resistor_SMD:R_0805_2012Metric_Pad1.20x1.40mm_HandSolder, F.Cu at (274.9, 92.0)
- added R13: 1K, Resistor_SMD:R_0805_2012Metric_Pad1.20x1.40mm_HandSolder, F.Cu at (297.1, 92.1)
- added R14: 10K, Resistor_SMD:R_0805_2012Metric_Pad1.20x1.40mm_HandSolder, F.Cu at (316.8, 92.0)
- added R15: 1K, Resistor_SMD:R_0805_2012Metric_Pad1.20x1.40mm_HandSolder, F.Cu at (339.0, 92.1)
- added R16: 10K, Resistor_SMD:R_0805_2012Metric_Pad1.20x1.40mm_HandSolder, F.Cu at (358.7, 92.0)
- added R3: 1K, Resistor_SMD:R_0805_2012Metric_Pad1.20x1.40mm_HandSolder, F.Cu at (93.0, 91.4)
- added R4: 10K, Resistor_SMD:R_0805_2012Metric_Pad1.20x1.40mm_HandSolder, F.Cu at (112.7, 91.3)
- added R5: 1K, Resistor_SMD:R_0805_2012Metric_Pad1.20x1.40mm_HandSolder, F.Cu at (128.4, 91.4)
- added R6: 10K, Resistor_SMD:R_0805_2012Metric_Pad1.20x1.40mm_HandSolder, F.Cu at (148.1, 91.3)
- added R7: 1K, Resistor_SMD:R_0805_2012Metric_Pad1.20x1.40mm_HandSolder, F.Cu at (168.8, 92.1)
- added R8: 10K, Resistor_SMD:R_0805_2012Metric_Pad1.20x1.40mm_HandSolder, F.Cu at (188.5, 92.0)
- added R9: 1K, Resistor_SMD:R_0805_2012Metric_Pad1.20x1.40mm_HandSolder, F.Cu at (212.0, 92.1)
- added U10: AT42QT1010, 0_sensor:AT42QT1010-TSGR_1, F.Cu at (350.5, 92.1)
- added U2: AT42QT1010, 0_sensor:AT42QT1010-TSGR_1, F.Cu at (104.6, 91.4)
- added U3: AT42QT1010, 0_sensor:AT42QT1010-TSGR_1, F.Cu at (140.0, 91.4)
- added U4: AT42QT1010, 0_sensor:AT42QT1010-TSGR_1, F.Cu at (180.3, 92.1)
- added U5: AT42QT1010, 0_sensor:AT42QT1010-TSGR_1, F.Cu at (223.5, 92.1)
- added U6: AT42QT1010, 0_sensor:AT42QT1010-TSGR_1, F.Cu at (266.7, 92.1)
- added U7: AT42QT1010, 0_sensor:AT42QT1010-TSGR_1, F.Cu at (308.6, 92.1)
- C1, C2: footprint Capacitor_SMD:C_1206_3216Metric_Pad1.33x1.80mm_HandSolder -> Capacitor_SMD:C_0805_2012Metric_Pad1.18x1.45mm_HandSolder
- D1: footprint LED_SMD:LED_1206_3216Metric_Pad1.42x1.75mm_HandSolder -> LED_SMD:LED_0805_2012Metric_Pad1.15x1.40mm_HandSolder
- R1, R2: footprint Resistor_SMD:R_1206_3216Metric_Pad1.30x1.75mm_HandSolder -> Resistor_SMD:R_0805_2012Metric_Pad1.20x1.40mm_HandSolder
- moved J2 250.6 mm to (383.9, 95.1), turned to 90 degrees
- moved JP9 162.5 mm to (366.5, 108.2), turned to 90 degrees
- moved JP10 161.6 mm to (366.5, 103.0), turned to -90 degrees
- moved U9 151.7 mm to (374.6, 105.4)
- moved J1 72.5 mm to (46.4, 106.8), turned to -90 degrees
- moved U8 16.0 mm to (203.4, 102.1)
- moved JP1 11.3 mm to (59.5, 89.5), turned to 0 degrees
- moved J4 4.32 mm to (80.8, 90.7)
- moved R1 4.30 mm to (56.0, 90.8), turned to -90 degrees
- moved C1 4.22 mm to (63.0, 90.9)
- moved C2 3.60 mm to (72.8, 90.7)
- moved R2 3.52 mm to (75.7, 90.7), turned to -90 degrees
- moved D1 3.30 mm to (59.6, 91.8), turned to 0 degrees
- moved U1 2.67 mm to (67.6, 90.8)
Connections:
- D1 pad 2: Net-(D1-A) -> TOUCH_8
- J1 pad 1: unconnected-(J1-Pin_1-Pad1) -> GND
- J1 pad 2: unconnected-(J1-Pin_2-Pad2) -> VCC
- J1 pad 3: unconnected-(J1-Pin_3-Pad3) -> CLK
- J1 pad 4: unconnected-(J1-Pin_4-Pad4) -> ~{LOAD}
- J1 pad 5: unconnected-(J1-Pin_5-Pad5) -> SERIAL_OUT
- J2 pad 1: unconnected-(J2-Pin_1-Pad1) -> GND
- J2 pad 2: unconnected-(J2-Pin_2-Pad2) -> VCC
- J2 pad 3: unconnected-(J2-Pin_3-Pad3) -> CLK_OUT
- J2 pad 4: unconnected-(J2-Pin_4-Pad4) -> LOAD_OUT
- J2 pad 5: unconnected-(J2-Pin_5-Pad5) -> SERIAL_IN
- JP1 pad 1: /Touch Sensor 1/TOUCH SENSE -> Net-(JP1-A)
- JP1 pad 2: Net-(D1-A) -> GND
- JP10 pad 1: unconnected-(JP10-A-Pad1) -> CLK_OUT
- JP10 pad 2: unconnected-(JP10-C-Pad2) -> CLK
- JP10 pad 3: unconnected-(JP10-B-Pad3) -> Net-(JP10-B)
- JP9 pad 1: unconnected-(JP9-A-Pad1) -> LOAD_OUT
- JP9 pad 2: unconnected-(JP9-C-Pad2) -> ~{LOAD}
- JP9 pad 3: unconnected-(JP9-B-Pad3) -> Net-(JP9-B)
- R1 pad 1: GND -> Net-(JP1-A)
- U1 pad 1: /Touch Sensor 1/TOUCH SENSE -> TOUCH_8
- U8 pad 1: unconnected-(U8-~{LD}-Pad1) -> ~{LOAD}
- U8 pad 10: unconnected-(U8-SER-Pad10) -> SERIAL_IN
- U8 pad 11: unconnected-(U8-A-Pad11) -> TOUCH_1
- U8 pad 12: unconnected-(U8-B-Pad12) -> TOUCH_2
- U8 pad 13: unconnected-(U8-C-Pad13) -> TOUCH_3
- U8 pad 14: unconnected-(U8-D-Pad14) -> TOUCH_4
- U8 pad 15: unconnected-(U8-~{CE}-Pad15) -> GND
- U8 pad 16: unconnected-(U8-VCC-Pad16) -> VCC
- U8 pad 2: unconnected-(U8-CLK-Pad2) -> CLK
- U8 pad 3: unconnected-(U8-E-Pad3) -> TOUCH_5
- U8 pad 4: unconnected-(U8-F-Pad4) -> TOUCH_6
- U8 pad 5: unconnected-(U8-G-Pad5) -> TOUCH_7
- U8 pad 6: unconnected-(U8-H-Pad6) -> TOUCH_8
- U8 pad 8: unconnected-(U8-GND-Pad8) -> GND
- U8 pad 9: unconnected-(U8-QH-Pad9) -> SERIAL_OUT
- U9 pad 1: unconnected-(U9-1A-Pad1) -> Net-(JP10-B)
- U9 pad 2: unconnected-(U9-GND-Pad2) -> GND
- U9 pad 3: unconnected-(U9-2A-Pad3) -> Net-(JP9-B)
- U9 pad 4: unconnected-(U9-2Y-Pad4) -> LOAD_OUT
- U9 pad 5: unconnected-(U9-VCC-Pad5) -> VCC
- U9 pad 6: unconnected-(U9-1Y-Pad6) -> CLK_OUT
Routing:
- net SERIAL_OUT: track 0.00 -> 196.7 mm
- net CLK: track 0.00 -> 188.5 mm
- net SERIAL_IN: track 0.00 -> 181.8 mm
- net ~{LOAD}: track 0.00 -> 174.3 mm
- net TOUCH_1: track 0.00 -> 154.1 mm
- net TOUCH_8: track 0.00 -> 146.3 mm
- net TOUCH_2: track 0.00 -> 113.3 mm
- net TOUCH_7: track 0.00 -> 108.4 mm
- net TOUCH_6: track 0.00 -> 72.2 mm
- net TOUCH_3: track 0.00 -> 69.5 mm
- net VCC: track 4.04 -> 37.8 mm
- net TOUCH_5: track 0.00 -> 31.8 mm
- net TOUCH_4: track 0.00 -> 25.2 mm
- net CLK_OUT: track 0.00 -> 21.0 mm
- net LOAD_OUT: track 0.00 -> 20.5 mm
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