File: Hardware/GVH_InteractiveCounter/GVH_InteractiveCounter.kicad_pcb (KiCad board)
At the start: 2 copper layers, 304.8 x 25.4 mm, 88 parts, among them J1 Molex Micro-Fit, J10 Electrode, J11 Electrode, J12 Conn_01x01, J13 Conn_01x01, J14 Conn_01x01, J15 Conn_01x01, J16 Conn_01x01, J17 Conn_01x01, J18 Conn_01x01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

Commit message: Finished another layout. This is probably the one.
Also  finished the touch pad layouts
Parts:
- J10, J11, J4, J5, J6, J7, J8, J9: footprint Connector_Pin:Pin_D1.3mm_L11.0mm_LooseFit -> Connector_Pin:Pin_D1.0mm_L10.0mm
- JP16, JP17: footprint Jumper:SolderJumper-2_P1.3mm_Open_Pad1.0x1.5mm -> Jumper:SolderJumper-2_P1.3mm_Open_RoundedPad1.0x1.5mm
- moved J13 169.6 mm to (247.3, 53.2)
- moved J18 139.2 mm to (174.2, 53.1)
- moved J15 98.2 mm to (252.0, 53.2)
- moved J17 96.4 mm to (327.7, 53.5)
- moved J16 73.9 mm to (169.6, 53.1)
- moved J14 72.1 mm to (92.8, 53.0)
- moved JP11 59.7 mm to (130.8, 53.1), turned to 180 degrees
- moved C19 59.1 mm to (138.0, 56.6)
- moved U11 54.0 mm to (133.3, 56.7), turned to 180 degrees
- moved C20 53.6 mm to (123.4, 56.6)
- moved C15 51.4 mm to (349.6, 56.2), turned to 180 degrees
- moved R16 50.5 mm to (356.7, 53.1), turned to -90 degrees
- moved C14 50.4 mm to (316.6, 57.1), turned to 90 degrees
- moved R14 50.0 mm to (316.6, 53.1)
- moved U10 49.9 mm to (353.7, 57.3), turned to 90 degrees
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Routing:
- net LOAD_OUT: track 265.9 -> 123.9 mm, vias 4 -> 1
- net VCC: track 377.1 -> 302.3 mm
- net +5V: track 399.4 -> 368.1 mm, vias 9 -> 13
- net TOUCH_8: track 139.1 -> 154.5 mm, vias 0 -> 2
- net CLK_OUT: track 258.4 -> 270.9 mm, vias 2 -> 0
- net GND: track 11.7 -> 0.00 mm
- net SERIAL_IN: track 147.2 -> 156.3 mm
- net Net-(JP14-A): track 14.9 -> 22.7 mm
- net TOUCH_7: track 121.4 -> 114.8 mm
- net CLK: track 21.8 -> 15.4 mm
- net Net-(D8-A): track 8.92 -> 3.58 mm
- net TOUCH_5: track 38.9 -> 33.9 mm
- net ~{LOAD}: track 25.7 -> 30.3 mm
- net TOUCH_2: track 104.3 -> 108.5 mm, vias 3 -> 2
- net TOUCH_1: track 144.4 -> 147.8 mm, vias 3 -> 2
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- removed copper zone on B.Cu, net GND
- removed copper zone on F.Cu, net GND
Other:
- board size 304.8 x 25.4 mm -> 317.5 x 25.4 mm
- board text removed: "IN"
- board text removed: "OUT"
