File: Hardware/GVH_InteractiveCounter/GVH_InteractiveCounter.kicad_pcb (KiCad board)
At the start: 2 copper layers, 317.5 x 25.4 mm, 88 parts, among them J1 Molex Micro-Fit, J10 Electrode, J11 Electrode, J12 Conn_01x01, J13 Conn_01x01, J14 Conn_01x01, J15 Conn_01x01, J16 Conn_01x01, J17 Conn_01x01, J18 Conn_01x01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

Commit message: Layouts done and ordered.
Parts:
- added G***: LOGO, 0_logo:MW_Mark_0.50inch, F.Cu at (291.3, 64.4)
- added G***: LOGO, 0_logo:MW_Logo_Horizontal_2.0inch, B.Cu at (287.4, 61.0)
- added G***: LOGO, 0_logo:UL_Mark_15mm_JLC_Single_Layer, B.Cu at (84.1, 73.2)
- added REF**: GVH_Cloak_Figure, 0_logo:GVH_Cloak_Figure, B.Cu at (171.7, 63.4)
- JP14, JP15: footprint Jumper:SolderJumper-3_P1.3mm_Open_RoundedPad1.0x1.5mm_NumberLabels -> Jumper:SolderJumper-3_P1.3mm_Bridged12_RoundedPad1.0x1.5mm
- U11: footprint Package_TO_SOT_THT:TO-220-3_Horizontal_TabDown -> Package_TO_SOT_SMD:TO-252-2
- moved C20 6.25 mm to (128.4, 52.8)
- moved U11 4.48 mm to (131.7, 60.8), turned to -90 degrees
- moved JP11 2.93 mm to (131.7, 55.9)
- moved C22 2.75 mm to (93.1, 68.3), turned to 90 degrees
- moved C17 2.35 mm to (210.7, 58.8), turned to 180 degrees
- moved C19 1.17 mm to (137.3, 55.8)
- moved J1 0.29 mm to (77.1, 67.0)
- moved J2 0.29 mm to (342.5, 67.0)
- turned JP14 to 90 degrees
- turned JP15 to 0 degrees
Connections:
- JP16 pad 1: Net-(JP14-A) -> Net-(JP14-B)
- JP17 pad 1: Net-(JP15-A) -> Net-(JP15-B)
- R17 pad 2: Net-(JP14-A) -> Net-(JP14-B)
- R18 pad 2: Net-(JP15-A) -> Net-(JP15-B)
- U13 pad 1: Net-(JP14-B) -> Net-(JP14-A)
- U13 pad 3: Net-(JP15-B) -> Net-(JP15-A)
- U13 pad 4: Net-(JP15-A) -> Net-(JP15-B)
- U13 pad 6: Net-(JP14-A) -> Net-(JP14-B)
Routing:
- net LOAD_OUT: track 132.2 -> 280.5 mm
- net GND: track 0.00 -> 53.0 mm, vias 0 -> 39
- net Net-(JP14-B): track 3.39 -> 24.8 mm
- net Net-(JP14-A): track 24.8 -> 3.39 mm
- net +5V: track 368.3 -> 382.5 mm, vias 13 -> 20
- net VCC: track 304.0 -> 294.4 mm
- net Net-(JP15-B): track 3.64 -> 12.0 mm
- net Net-(JP15-A): track 12.0 -> 3.64 mm
- net CLK_OUT: track 269.3 -> 267.9 mm
- net TOUCH_8: track 154.5 -> 153.4 mm
- net TOUCH_7: track 114.8 -> 115.6 mm
- net (no net): vias 1 -> 0
- added copper zone on B.Cu, net GND
- added copper zone on F.Cu, net GND
Other:
- board text added: "GND"
- board text added: "GVH • Cap Touch Counter Sensor Board • V0.1 Daniel Bornhorst • 12/2024"
- board text added: "IN"
- board text added: "IN Ser← Clk→ LD→"
- board text added: "OUT"
- board text added: "OUT Ser → Clk ← LD ←"
