File: Hardware/GVH_InteractiveCounter/GVH_InteractiveCounter_Layout_Pass3.kicad_pcb (KiCad board)
At the start: 2 copper layers, 317.5 x 25.4 mm, 88 parts, among them J1 Molex Micro-Fit, J10 Electrode, J11 Electrode, J12 Conn_01x01, J13 Conn_01x01, J14 Conn_01x01, J15 Conn_01x01, J16 Conn_01x01, J17 Conn_01x01, J18 Conn_01x01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

Commit message: Layouts done and ordered.
Routing:
- added copper zone on B.Cu, net GND
- added copper zone on F.Cu, net GND
Changed lines of the file:
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@@
+    )
+  )
+  (zone (net 2) (net_name "GND") (layers "F&B.Cu") (hatch edge 0.5)
+    (connect_pads (clearance 0.5))
+    (min_thickness 0.25) (filled_areas_thickness no)
+    (fill yes (thermal_gap 0.5) (thermal_bridge_width 0.5))
+    (polygon
+      (pts
+        (xy 60.325 50.8)
+        (xy 358.775 50.8)
+        (xy 358.775 76.2)
+        (xy 60.325 76.2)
+      )
     )
   )
