File: Hardware/GVH_CounterController/IO_Level_Shift.kicad_sch (KiCad schematic)
At the start: 5 parts, among them J4 Molex Micro-Fit 5pos, U4 74LVC2G125DC,125, U6 74LVC2G125DC,125

Commit message: Added Mosfet fan controller to CounterController Schematic
Connections:
- net CLK: now also U4.5 (2A); no longer U4.2 (1A)
- net LOAD: now also U4.2 (1A); no longer U4.5 (2A)
- net at U4.3 (2Y): now also J4.3 (Pin_3); no longer J4.4 (Pin_4)
- net at U4.6 (1Y): now also J4.4 (Pin_4); no longer J4.3 (Pin_3)
Changed lines of the file:
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@@
     (stroke (width 0) (type default))
   )
-  (wire (pts (xy 157.48 73.66) (xy 157.48 66.04))
+  (wire (pts (xy 185.928 73.66) (xy 185.928 63.5))
     (stroke (width 0) (type default))
   )
@@
     (stroke (width 0) (type default))
   )
-  (wire (pts (xy 68.58 73.66) (xy 130.81 73.66))
-    (stroke (width 0) (type default))
-  )
   (wire (pts (xy 128.27 53.34) (xy 139.7 53.34))
     (stroke (width 0) (type default))
@@
     (stroke (width 0) (type default))
   )
-  (wire (pts (xy 157.48 66.04) (xy 187.96 66.04))
+  (wire (pts (xy 166.37 63.5) (xy 148.59 63.5))
+    (stroke (width 0) (type default))
+  )
+  (wire (pts (xy 185.928 63.5) (xy 187.96 63.5))
     (stroke (width 0) (type default))
   )
@@
     (stroke (width 0) (type default))
   )
-  (wire (pts (xy 148.59 73.66) (xy 157.48 73.66))
+  (wire (pts (xy 68.326 73.66) (xy 130.81 73.66))
     (stroke (width 0) (type default))
   )
@@
     (stroke (width 0) (type default))
   )
+  (wire (pts (xy 148.59 73.66) (xy 185.928 73.66))
+    (stroke (width 0) (type default))
+  )
   (wire (pts (xy 128.27 82.55) (xy 139.7 82.55))
     (stroke (width 0) (type default))
@@
     (stroke (width 0) (type default))
   )
-  (wire (pts (xy 187.96 63.5) (xy 148.59 63.5))
+  (wire (pts (xy 187.96 66.04) (xy 166.37 66.04))
     (stroke (width 0) (type default))
   )
@@
   )
   (wire (pts (xy 128.27 63.5) (xy 128.27 71.12))
+    (stroke (width 0) (type default))
+  )
+  (wire (pts (xy 166.37 66.04) (xy 166.37 63.5))
     (stroke (width 0) (type default))
   )
@@
     (stroke (width 0) (type default))
   )
-  (hierarchical_label "LOAD" (shape input) (at 68.58 73.66 180) (fields_autoplaced)
+  (hierarchical_label "LOAD" (shape input) (at 68.58 66.04 180) (fields_autoplaced)
     (effects (font (size 1.27 1.27)) (justify right))
   )
@@
     (effects (font (size 1.27 1.27)) (justify right))
   )
-  (hierarchical_label "CLK" (shape input) (at 68.58 66.04 180) (fields_autoplaced)
+  (hierarchical_label "CLK" (shape input) (at 68.326 73.66 180) (fields_autoplaced)
     (effects (font (size 1.27 1.27)) (justify right))
   )
+  (netclass_flag "" (length 1.27) (shape dot) (at 128.27 53.34 0) (fields_autoplaced)
+    (effects (font (size 1.27 1.27)) (justify left bottom))
+    (property "Netclass" "Default" (at 128.9685 52.07 0)
+      (effects (font (size 1.27 1.27) italic) (justify left) hide)
+    )
+  )
   (symbol (lib_id "KTX-MultiPCB:74AHCT2G125") (at 139.7 68.58 0) (unit 1)

Commit message: Added header for two board stack design
This will allow the fans to be connected horizontally
Parts:
- removed J4: Molex Micro-Fit 5pos, 0_connector:MOLEX_MICROFIT-RA-5POS_436500500, symbol 0_connector:Molex Micro-Fit 5pos
Connections:
- net SERIAL_IN: now also U6.2 (1A); no longer U6.6 (1Y)
- net CLK_OUT: now reaches U4.3 (2Y)
- net LOAD_OUT: now reaches U4.6 (1Y)
- new net SERIAL: U6.6 (1Y)
