File: Hardware/GVH_CounterController/GVH_CounterContoller.kicad_sch (KiCad schematic)
At the start: 31 parts, among them J1 Molex Ultra-Fit, J2 WIZnet_J1B1211CCD_RJ45, J3 Barrel jack, SW1 SW_DIP_x02, SW2 SW_MEC_5G, U1 R-78B5.0-2.0, U2 Teensy4.1, U3 R-78B3.3-2.0, U5 DS18B20_

Commit message: Counter Controller PCB - Added IO Level Shifter Sheet, Updated from Template
Parts:
- removed C10: 0.1uF, Capacitor_SMD:C_0805_2012Metric, symbol Device:C_Small
- removed C4, C6: 10uF, Capacitor_SMD:C_1206_3216Metric, symbol Device:C
- removed C5: 4.7uF, Capacitor_SMD:C_1206_3216Metric, symbol Device:C
- removed D1: Reverse Protection Diode, Package_TO_SOT_SMD:TO-252-2_TabPin1, symbol Device:D
- removed F1: Fuse, MeowWolf_Devices:Fuseholder_5x20mm_Littelfuse_01110501Z, symbol Device:Fuse
- removed J1: Molex Ultra-Fit, 0_connector:MOLEX_ULTRAFIT-RA-2POS_1723104102, symbol 0_connector:Molex Ultra-Fit 2pos IN
- removed J2: WIZnet_J1B1211CCD_RJ45, 0_connector:WIZnet_J1B1211CCD_RJ45, symbol 0_connector:WIZnet_J1B1211CCD_RJ45
- removed J3: Barrel jack, Connector_BarrelJack:BarrelJack_Horizontal, symbol Connector:Barrel_Jack_Switch
- removed L2: 10uH, Inductor_SMD:L_Changjiang_FNR6045S, symbol Device:L
- removed U2: Teensy4.1, 0_microcontroller:Teensy41_ethernet_only, symbol 0_microcontroller:Teensy4.1
- removed U3: R-78B3.3-2.0, MeowWolf_Devices:DC-DC_CONVERTER_R-78E_R-78B, symbol MeowWolf_Devices:R-78E5.0-1.0
- added C13, C17: 10uF, Capacitor_SMD:C_0805_2012Metric, symbol Device:C_Small
- added C18: 0.1uF, Capacitor_SMD:C_0805_2012Metric, symbol Device:C_Small
- added D7: PMEG045V100EPD, Package_TO_SOT_SMD:Nexperia_CFP15_SOT-1289, symbol Diode:PMEG045V100EPD
- added D8: 1N4148, Diode_SMD:D_SOD-323, symbol Device:D_Small
- added D9: RED LED, LED_SMD:LED_0603_1608Metric, symbol Device:LED
- added J4: Molex Ultra-Fit, 0_connector:MOLEX_ULTRAFIT-RA-2POS_1723104102, symbol 0_connector:Molex Ultra-Fit 2pos IN
- added J5: Barrel jack, Connector_BarrelJack:BarrelJack_Horizontal, symbol Connector:Barrel_Jack_Switch
- added J6: WIZnet_J1B1211CCD_RJ45, 0_connector:WIZnet_J1B1211CCD_RJ45, symbol 0_connector:WIZnet_J1B1211CCD_RJ45
- added JP1: SolderJumper_2_Open, Jumper:SolderJumper-2_P1.3mm_Open_RoundedPad1.0x1.5mm, symbol Jumper:SolderJumper_2_Open
- added K1: Relay_DPDT, Relay_THT:Relay_DPDT_Kemet_EC2, symbol Relay:EC2-3NU
- added Q1: MBT2222, Package_TO_SOT_SMD:SOT-23-3, symbol Device:Q_NPN_BEC
- added R4, R7: 10k, Resistor_SMD:R_0603_1608Metric, symbol Device:R_Small
- added R5, R6: 1k, Resistor_SMD:R_0603_1608Metric, symbol Device:R_Small
- added U4: RT9080-3.3, Package_TO_SOT_SMD:SOT-23-5, symbol 0_power:RT9080-3.3
- added U8: Teensy4.1, 0_microcontroller:Teensy41_ethernet_only, symbol 0_microcontroller:Teensy4.1_ethernet_only
- C2: value 4.7uF -> 10uF; Digikey P/N 1276-2789-1-ND -> 1276-6767-1-ND; Digikey Page https://www.digikey.com/en/products/detail/samsung-electro-mechanics/CL31B475KBHNNNE/3888447?s=N4IgTCBcDaIMIBkDMBGAQgFgOwFYDSaAEgHKkCiIAugL5A -> https://www.digikey.com/en/products/detail/samsung-electro-mechanics/CL31B106KBHNNNE/5961251?s=N4IgTCBcDaIMIBkDMBGAQigDANgNJoAkA5EgURAF0BfIA; LCSC C51205 -> C89632; MPN CL31B475KBHNNNE -> CL31B106KBHNNNE
- L1: value 10uH -> 12uH; footprint Inductor_SMD:L_Changjiang_FNR6045S -> Inductor_SMD:L_Changjiang_FNR4030S; LCSC C2827404 -> C167880; MPN SNR6045TYD100M -> FNR4030S120MT; Manufacturer SOREDE -> Changjiang Microelectronics Tech; Package 6045 SMD,6x6m -> SMD,4x4mm
- R1: value 560 -> 1k; LCSC C114629 -> C22548; MPN RC0603FR-07560RL -> RC0603FR-071KL
- R2: value 220 -> 1k; LCSC C107696 -> C22548; MPN RC0603FR-07220RL -> RC0603FR-071KL
- U1: value R-78B5.0-2.0 -> R-78E5.0-1.0; footprint MeowWolf_Devices:DC-DC_CONVERTER_R-78E_R-78B -> MeowWolf_Devices:DC-DC_CONVERTER_R-78E5; Digikey P/N 945-3042-ND -> 945-2201-ND; Digikey Page https://www.digikey.com/en/products/detail/recom-power/R-78B5-0-2-0/6677084 -> https://www.digikey.com/en/products/detail/recom-power/R-78E5-0-1-0/4930585; MPN R-78B5.0-2.0 -> R-78E5.0-1.0
Connections:
- net +12V: now also D7.3 (K), JP1.2 (B), K1.4
- net +3.3V: now also C13.1, D8.1 (K), K1.1, R5.1, U4.5 (OUT)
- net +5V: now also C17.1, R4.2, U4.1 (IN), U8.48 (VIN)
- net GND: now also C13.2, C17.2, C18.1, J4.1 (Pin_1), J5.2, J5.3, J6.8, J6.9, Q1.2 (E), R7.1, U4.2 (GND), U8.1 (GND), U8.34 (GND), U8.47 (GND), U8.64 (GND)
- new net: D8.2 (A), D9.1 (K), K1.12, Q1.3 (C)
- new net: D7.1 (A), D7.2 (A), J4.2 (Pin_2), J5.1
- new net: Q1.1 (B), R6.2, R7.2
- new net: R4.1, U4.3 (EN)
- new net: J6.4, U8.60 (R+)
- new net: J6.10, U8.61 (LED)
- new net: J6.3, U8.62 (T-)
- new net: J6.1, U8.63 (T+)
- new net: J6.6, U8.65 (R-)
- new net: D9.2 (A), R5.2
- new net: C18.2, J6.2, J6.5
- new net +12V_ISO: JP1.1 (A), K1.3
- new net IO_Level_Shift/CLK: U8.45 (23_A9_CRX1_MCLK1)
- new net IO_Level_Shift/LOAD: U8.44 (22_A8_CTX1)
- new net IO_Level_Shift/SERIAL_IN: U8.43 (21_A7_RX5_BCLK1)
- new net IO_Level_Shift1/CLK: U8.39 (17_A3_TX4_SDA1)
- new net IO_Level_Shift1/LOAD: U8.38 (16_A2_RX4_SCL1)
- new net IO_Level_Shift1/SERIAL_IN: U8.37 (15_A1_RX3_SPDIF_IN)
- new net IO_Level_Shift2/CLK: U8.33 (41_A17)
- new net IO_Level_Shift2/LOAD: U8.32 (40_A16)
- new net IO_Level_Shift2/SERIAL_IN: U8.31 (39_MISO1_OUT1A)
- new net IO_Level_Shift3/CLK: U8.27 (35_TX8)
- new net IO_Level_Shift3/LOAD: U8.26 (34_RX8)
- new net IO_Level_Shift3/SERIAL_IN: U8.25 (33_MCLK2)
- new net TOUCH_RESET: R6.1
- no-connect marks 15 -> 3
Other:
- removed sheet Input_Output
- added sheet IO_Level_Shift (IO_Level_Shift.kicad_sch)
- added sheet IO_Level_Shift1 (IO_Level_Shift.kicad_sch)
- added sheet IO_Level_Shift2 (IO_Level_Shift.kicad_sch)
- added sheet IO_Level_Shift3 (IO_Level_Shift.kicad_sch)
- note added: "5V to 3.3V"
- note added: "Relay Bypass"
- note added: "Touch Reset Relay"
- note removed: "12V to 3.3V"
- note removed: "ADD RELAY TO RESET TOUCH SENSORS"
- moved on the sheet: D4, R3, U5

Commit message: Bump
Parts:
- renumbered C17 to C4, C13 to C5, C18 to C6, D7 to D1, D9 to D2, D8 to D3, D2 to D4, D3 to D5, D4 to D6, J4 to J1, J5 to J2, J6 to J3, R5 to R1, R6 to R2, R7 to R3, R1 to R5, R2 to R6, R3 to R7, U8 to U1, U1 to U2, U4 to U3, U5 to U4
Other:
- moved on the sheet: D6, R7, U4

Commit message: Added Mosfet fan controller to CounterController Schematic
Parts:
- removed J2: Barrel jack, Connector_BarrelJack:BarrelJack_Horizontal, symbol Connector:Barrel_Jack_Switch
- added C16: 0.1uF, Capacitor_SMD:C_0402_1005Metric, symbol Device:C_Small
- added D7, D8: PMEG10030, Diode_SMD:D_SOD-128, symbol Device:D
- added J10, J11, J12, J2, J8, J9: Molex Micro-Fit 2pos, 0_connector:MOLEX_MICROFIT-VERT-2POS_436500215, symbol 0_connector:Molex Micro-Fit 2pos
- added J13: Molex Micro-Fit 3pos, 0_connector:MOLEX_MICROFIT-VERT-3POS_436500315, symbol 0_connector:Molex Micro-Fit 3pos Vert
- added JP2: SolderJumper_2_Bridged, Jumper:SolderJumper-2_P1.3mm_Bridged_RoundedPad1.0x1.5mm, symbol Jumper:SolderJumper_2_Bridged
- added Q2, Q3: AO3406, Package_TO_SOT_SMD:SOT-23, symbol Transistor_FET:AO3400A
- added R10, R8: 100R, Resistor_SMD:R_0603_1608Metric, symbol Device:R_Small
- added R11, R12: 10k, Resistor_SMD:R_0603_1608Metric, symbol Device:R_Small
- added R9: 4.7k, Resistor_SMD:R_0603_1608Metric, symbol Device:R
- added U14: SN74LVC2G17, Package_TO_SOT_SMD:SOT-23-6, symbol 0_integrated_circuits:SN74LVC2G17
- D1: Package (none) -> TO-277
- JP1: now left out of the parts list
Connections:
- net +12V: now also D7.1 (K), D8.1 (K), J10.2 (Pin_2), J11.2 (Pin_2), J12.2 (Pin_2), J2.2 (Pin_2), J8.2 (Pin_2), J9.2 (Pin_2)
- net +3.3V: now also J13.2 (Pin_2), JP2.1 (A), R9.2; no longer D5.2 (A)
- net +5V: now also C16.1, U14.5 (VCC)
- net GND: now also C16.2, J13.1 (Pin_1), Q2.2 (S), Q3.2 (S), R11.1, R12.1, U14.2 (GND)
- net IO_Level_Shift2/CLK: no longer U1.33 (41_A17)
- net IO_Level_Shift2/LOAD: no longer U1.32 (40_A16)
- net IO_Level_Shift2/SERIAL_IN: no longer U1.31 (39_MISO1_OUT1A)
- net IO_Level_Shift3/CLK: no longer U1.27 (35_TX8)
- net IO_Level_Shift3/LOAD: no longer U1.26 (34_RX8)
- net IO_Level_Shift3/SERIAL_IN: no longer U1.25 (33_MCLK2)
- net SER_0: now reaches U1.12 (10_CS_MQSR)
- net CLK_0: now reaches U1.13 (11_MOSI_CTX1)
- net LOAD_0: now reaches U1.14 (12_MISO_MQSL)
- net SER_1: now reaches U1.20 (28_RX7)
- net CLK_1: now reaches U1.21 (29_TX7)
- net LOAD_1: now reaches U1.22 (30_CRX3)
- net DIP1 renamed DIP_0
- net DIP2 renamed DIP_1
- net IO_Level_Shift/CLK: no longer names the net of U1.45 (23_A9_CRX1_MCLK1)
- net IO_Level_Shift/LOAD: no longer names the net of U1.44 (22_A8_CTX1)
- net IO_Level_Shift/SERIAL_IN: no longer names the net of U1.43 (21_A7_RX5_BCLK1)
- net IO_Level_Shift1/CLK: no longer names the net of U1.39 (17_A3_TX4_SDA1)
- net IO_Level_Shift1/LOAD: no longer names the net of U1.38 (16_A2_RX4_SCL1)
- net IO_Level_Shift1/SERIAL_IN: no longer names the net of U1.37 (15_A1_RX3_SPDIF_IN)
- net TEMP_SENS1 renamed TEMP_SENS_0
- new net: Q2.1 (G), R8.2
- new net: D7.2 (A), J11.1 (Pin_1), J12.1 (Pin_1), Q2.3 (D)
- new net: R10.1, R11.2, U14.4 (2Y)
- new net: R12.2, R8.1, U14.6 (1Y)
- new net: D8.2 (A), J10.1 (Pin_1), J2.1 (Pin_1), J8.1 (Pin_1), J9.1 (Pin_1), Q3.3 (D)
- new net: D5.2 (A), JP2.2 (B)
- new net: Q3.1 (G), R10.2
- new net FAN_0: U14.1 (1A)
- new net FAN_1: U14.3 (2A)
- new net TEMP_SENS_1: J13.3 (Pin_3), R9.1
Other:
- note added: "RED LED"
- note removed: "3.3V RED LED"
- moved on the sheet: D5, D6, R6, R7, U4

Commit message: Checkpoint before rerouting the power supply
Connections:
- net BUTTON: no longer SW2.2 (B)
- net GND: no longer SW2.4 (B)
Changed lines of the file:
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@@
       (effects (font (size 1.27 1.27)) hide)
     )
-    (property "Datasheet" "" (at 53.34 172.72 0)
+    (property "Datasheet" "https://omronfs.omron.com/en_US/ecb/products/pdf/en-b3f.pdf" (at 53.34 172.72 0)
       (effects (font (size 1.27 1.27)) hide)
     )
@@
       (effects (font (size 1.27 1.27)) hide)
     )
-    (property "Manufacturer" "Omron Electronics Inc-EMC Div" (at 53.34 177.8 0)
-      (effects (font (size 1.27 1.27)) hide)
-    )
-    (property "Digikey P/N" "SW402-ND" (at 53.34 177.8 0)
-      (effects (font (size 1.27 1.27)) hide)
-    )
-    (property "Digikey Page" "https://www.digikey.com/en/products/detail/omron-electronics-inc-emc-div/B3F-1020/44059" (at 53.34 177.8 0)
-      (effects (font (size 1.27 1.27)) hide)
-    )
-    (property "MPN" "B3F-1020" (at 53.34 177.8 0)
-      (effects (font (size 1.27 1.27)) hide)
-    )
-    (property "Description" "Tactile Switch SPST-NO Top Actuated Through Hole" (at 53.34 177.8 0)
-      (effects (font (size 1.27 1.27)) hide)
-    )
-    (pin "2")
-    (pin "4")
+    (property "Manufacturer" "Omron Electronics Inc-EMC Div" (at 53.086 182.88 0)
+      (effects (font (size 1.27 1.27)) hide)
+    )
+    (property "Digikey P/N" "SW402-ND" (at 52.324 186.944 0)
+      (effects (font (size 1.27 1.27)) hide)
+    )
+    (property "Digikey Page" "https://www.digikey.com/en/products/detail/omron-electronics-inc-emc-div/B3F-1020/44059" (at 53.34 180.594 0)
+      (effects (font (size 1.27 1.27)) hide)
+    )
+    (property "MPN" "B3F-1020" (at 53.086 179.324 0)
+      (effects (font (size 1.27 1.27)) hide)
+    )
+    (property "Description" "Tactile Switch SPST-NO Top Actuated Through Hole" (at 53.086 184.658 0)
+      (effects (font (size 1.27 1.27)) hide)
+    )
     (pin "1")
     (pin "2")
@@
     )
   )
+  (symbol (lib_id "power:GND") (at 58.42 180.34 0) (unit 1)
+    (in_bom yes) (on_board yes) (dnp no)
+    (property "Reference" "#PWR021" (at 58.42 186.69 0)
+      (effects (font (size 1.27 1.27)) hide)
+    )
+    (property "Value" "GND" (at 58.547 184.7342 0)
+      (effects (font (size 1.27 1.27)))
+    )
+    (property "Footprint" "" (at 58.42 180.34 0)
+      (effects (font (size 1.27 1.27)) hide)
+    )
+    (property "Datasheet" "" (at 58.42 180.34 0)
+      (effects (font (size 1.27 1.27)) hide)
+    )
+    (pin "1")
+    (instances
+      (project "GVH_CounterContoller"
+        (path "/2012002c-7ba5-4575-b93c-d8b37d21ac31"
+          (reference "#PWR021") (unit 1)
+        )
+      )
+      (project "KTX-MultiPCB"
+        (path "/aa56e0db-dcb9-4815-a5d6-811d95d9cf15/00000000-0000-0000-0000-00006034b2d9"
+          (reference "#PWR?") (unit 1)
+        )
+        (path "/aa56e0db-dcb9-4815-a5d6-811d95d9cf15"
+          (reference "#PWR04") (unit 1)
+        )
+      )
+    )
+  )
   (symbol (lib_id "Device:R_Small") (at 295.91 74.93 90) (unit 1)
     (in_bom yes) (on_board yes) (dnp no)
@@
         )
       )
-    )
-  )
-  (symbol (lib_id "power:GND") (at 58.42 180.34 0) (unit 1)
-    (in_bom yes) (on_board yes) (dnp no) (fields_autoplaced)
-    (property "Reference" "#PWR021" (at 58.42 186.69 0)
-      (effects (font (size 1.27 1.27)) hide)
-    )
-    (property "Value" "GND" (at 58.42 185.42 0)
-      (effects (font (size 1.27 1.27)))
-    )
-    (property "Footprint" "" (at 58.42 180.34 0)
-      (effects (font (size 1.27 1.27)) hide)
-    )
-    (property "Datasheet" "" (at 58.42 180.34 0)
-      (effects (font (size 1.27 1.27)) hide)
-    )
-    (pin "1")
-    (instances
-      (project "GVH_CounterContoller"
-        (path "/2012002c-7ba5-4575-b93c-d8b37d21ac31"
-          (reference "#PWR021") (unit 1)
-        )
-      )
-      (project "GVH-SwissArmyPCB"
-        (path "/38ccbc2b-e79d-43d1-80a7-cb797d9e77eb"
-          (reference "#PWR011") (unit 1)
-        )
-      )

Commit message: Added header for two board stack design
This will allow the fans to be connected horizontally
Parts:
- removed JP1: SolderJumper_2_Open, Jumper:SolderJumper-2_P1.3mm_Open_RoundedPad1.0x1.5mm, symbol Jumper:SolderJumper_2_Open
- removed Q2, Q3: AO3406, Package_TO_SOT_SMD:SOT-23, symbol Transistor_FET:AO3400A
- added C15, C17: 1uF, Capacitor_SMD:C_0603_1608Metric, symbol Device:C_Small
- added C18: 10uF, Capacitor_SMD:C_0805_2012Metric, symbol Device:C_Small
- added D9: Reverse Protection Diode, Package_TO_SOT_SMD:TO-252-2_TabPin1, symbol Device:D
- added F1: Fuse, MeowWolf_Devices:Fuseholder_2AG_5x15mm_Littelfuse_01110501Z, symbol Device:Fuse
- added J14: Molex Ultra-Fit, 0_connector:MOLEX_ULTRAFIT-RA-2POS_1723104102, symbol 0_connector:Molex Ultra-Fit 2pos IN
- added J15: Barrel jack, Connector_BarrelJack:BarrelJack_Horizontal, symbol Connector:Barrel_Jack_Switch
- added J16: Conn_02x08_Odd_Even, Connector_PinHeader_2.54mm:PinHeader_2x08_P2.54mm_Vertical, symbol Connector_Generic:Conn_02x08_Odd_Even
- added J4, J5: Molex Micro-Fit 5pos, 0_connector:MOLEX_MICROFIT-RA-5POS_436500500, symbol 0_connector:Molex Micro-Fit 5pos
- added SW3: SW_DIP_x02, Button_Switch_SMD:SW_DIP_SPSTx02_Slide_KingTek_DSHP02TS_W7.62mm_P1.27mm, symbol Switch:SW_DIP_x02
- added U13: TLV1117LV33, Package_TO_SOT_SMD:SOT-223, symbol Regulator_Linear:TLV1117-33
- added U15: AO4882, Package_SO:SOIC-8_3.9x4.9mm_P1.27mm, symbol 0_integrated_circuits:AO4882_Dual_Mosfet
- C4, C5: Digikey P/N (none) -> 1276-2891-1-ND; Digikey Page (none) -> https://www.digikey.com/en/products/detail/samsung-electro-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; MPN (none) -> CL21A106KAYNNNE; Manufacturer (none) -> Samsung Electro-Mechanics
- J13: footprint 0_connector:MOLEX_MICROFIT-VERT-3POS_436500315 -> 0_connector:MOLEX_MICROFIT-RA-3POS_436500300
Connections:
- net +12V: now also D9.1 (K), F1.1
- net +12V_ISO: now also J4.2 (Pin_2), J5.2 (Pin_2)
- net +3.3V: now also R1.2, C17.1, C18.1, U13.2 (VO); no longer R1.1
- net +5V: now also C15.1, U13.3 (VI)
- net GND: now also C15.2, C17.2, C18.2, D9.2 (A), J14.1 (Pin_1), J15.2, J15.3, J4.1 (Pin_1), J5.1 (Pin_1), U13.1 (GND), U15.1 (S), U15.3 (S)
- net at R8.2: now also U15.2 (G)
- net at D7.2 (A), J11.1 (Pin_1), J12.1 (Pin_1): now also U15.7 (D), U15.8 (D)
- net CLK_2: now reaches U1.27 (35_TX8)
- net LOAD_2: now reaches U1.28 (36_CS)
- net SER_2: now reaches U1.29 (37_CS)
- net at D8.2 (A), J10.1 (Pin_1), J2.1 (Pin_1)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: now also U15.5 (D), U15.6 (D)
- net at D2.2 (A): now also R1.1; no longer R1.2
- net at R10.2: now also U15.4 (G)
- new net: F1.2, J14.2 (Pin_2), J15.1
- new net IO_Level_Shift/CLK_OUT: J4.3 (Pin_3)
- new net IO_Level_Shift/LOAD_OUT: J4.4 (Pin_4)
- new net IO_Level_Shift/SERIAL_IN: J4.5 (Pin_5)
- new net IO_Level_Shift1/CLK_OUT: J5.3 (Pin_3)
- new net IO_Level_Shift1/LOAD_OUT: J5.4 (Pin_4)
- new net IO_Level_Shift1/SERIAL_IN: J5.5 (Pin_5)
Other:
- sheet IO_Level_Shift ports: added CLK_OUT, LOAD_OUT, SERIAL; removed none
- sheet IO_Level_Shift1 ports: added CLK_OUT, LOAD_OUT, SERIAL; removed none
- sheet IO_Level_Shift2 ports: added CLK_OUT, LOAD_OUT, SERIAL; removed none
- sheet IO_Level_Shift3 ports: added CLK_OUT, LOAD_OUT, SERIAL; removed none
- note added: "2Ch MOSFET Fan Controller"
- note added: "GND +12V CLK LOAD SERIAL"
- note removed: "Relay Bypass"
- moved on the sheet: C16, D2, D3, D7, D8, J10, J11, J12, J2, J8, J9, K1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

Commit message: Checkpoint before removing fan connectors
Connections:
- net +12V: now also J16.16 (Pin_16)
- net +12V_ISO: now also J16.15 (Pin_15)
- net +3.3V: now also J16.2 (Pin_2), R1.1; no longer R1.2
- net +5V: now also J16.1 (Pin_1)
- net BUTTON: now also SW2.2 (B), U1.4 (2_OUT2); no longer SW2.1 (A)
- net CLK_2: now also U1.26 (34_RX8); no longer U1.27 (35_TX8)
- net CLK_2_OUT: now also J16.13 (Pin_13)
- net CLK_3: now also U1.36 (14_A0_TX3_SPDIF_OUT)
- net CLK_3_OUT: now also J16.7 (Pin_7)
- net DIP_0: now also SW3.4, U1.2 (0_RX1_CRX2_CS1); no longer SW1.4
- net DIP_1: now also SW3.3, U1.3 (1_TX1_CTX2_MISO1); no longer SW1.3
- net GND: now also J16.12 (Pin_12), J16.14 (Pin_14), SW2.1 (A), SW3.1, SW3.2; no longer SW1.1, SW1.2, SW2.2 (B)
- net LD_2_OUT: now also J16.11 (Pin_11)
- net LD_3_OUT: now also J16.5 (Pin_5)
- net LOAD_2: now also U1.25 (33_MCLK2); no longer U1.28 (36_CS)
- net LOAD_3: now also U1.35 (13_SCK_LED)
- net SER_2: now also U1.27 (35_TX8); no longer U1.29 (37_CS)
- net SER_2_OUT: now also J16.9 (Pin_9)
- net SER_3: now also U1.37 (15_A1_RX3_SPDIF_IN)
- net SER_3_OUT: now also J16.3 (Pin_3)
- net at D2.2 (A): now also R1.2; no longer R1.1
Other:
- note added: "Class A EMI Filter"
- moved on the sheet: C15, C17, C18, D9, F1, J14, J15, R1, SW1, SW3, U13

Commit message: Noticed that voltage translators wont work 3-5v, changing that part
Parts:
- removed J10, J11, J12, J2, J8, J9: Molex Micro-Fit 2pos, 0_connector:MOLEX_MICROFIT-VERT-2POS_436500215, symbol 0_connector:Molex Micro-Fit 2pos
- added J2, J6, J7: Molex Micro-Fit 2pos, 0_connector:MOLEX_MICROFIT-VERT-2POS_436500215, symbol 0_connector:Molex Micro-Fit 2pos Vert
Connections:
- net +12V: now also J2.2 (Pin_2), J6.2 (Pin_2), J7.2 (Pin_2)
- net BUTTON: now also SW2.1 (A), U1.2 (0_RX1_CRX2_CS1); no longer SW2.2 (B), U1.4 (2_OUT2)
- net DIP_0: now also U1.3 (1_TX1_CTX2_MISO1); no longer U1.2 (0_RX1_CRX2_CS1)
- net DIP_1: now also U1.4 (2_OUT2); no longer U1.3 (1_TX1_CTX2_MISO1)
- net GND: now also SW2.2 (B); no longer SW2.1 (A)
- net STATUS_PIXEL: now also U1.45 (23_A9_CRX1_MCLK1)
- net FAN_PWR_1: now reaches D8.2 (A), U15.5 (D), U15.6 (D)
- net FAN_PWR_1: now also J6.1 (Pin_1), J7.1 (Pin_1)
- net FAN_PWR_0: now reaches D7.2 (A), U15.7 (D), U15.8 (D)
- net FAN_PWR_0: now also J2.1 (Pin_1)
- net FAN_0 renamed FAN_CTRL_0
- net FAN_1 renamed FAN_CTRL_1
Other:
- moved on the sheet: C16, D7, R10, R11, R12, R8, U14, U15

Commit message: Level shifting redesign complete
Parts:
- removed C18: 10uF, Capacitor_SMD:C_0805_2012Metric, symbol Device:C_Small
- removed J15: Barrel jack, Connector_BarrelJack:BarrelJack_Horizontal, symbol Connector:Barrel_Jack_Switch
- removed SW1: SW_DIP_x02, Button_Switch_THT:SW_DIP_SPSTx02_Slide_9.78x7.26mm_W7.62mm_P2.54mm, symbol Switch:SW_DIP_x02
- removed U13: TLV1117LV33, Package_TO_SOT_SMD:SOT-223, symbol Regulator_Linear:TLV1117-33
- added C1, C14, C16, C2, C6, C7: 0.1uF, Capacitor_SMD:C_0402_1005Metric, symbol Device:C_Small
- added U2: SN74LVC2T45, Package_SO:VSSOP-8_2.4x2.1mm_P0.5mm, symbol Logic_LevelTranslator:SN74LVC2T45DCUR
- added U5, U7, U8: SN74LVC2T45DCUR, Package_SO:VSSOP-8_2.4x2.1mm_P0.5mm, symbol Logic_LevelTranslator:SN74LVC2T45DCUR
- C15, C17: value 1uF -> 0.1uF; footprint Capacitor_SMD:C_0603_1608Metric -> Capacitor_SMD:C_0402_1005Metric; Digikey P/N (none) -> 1276-1001-1-ND; Digikey Page (none) -> https://www.digikey.com/en/products/detail/samsung-electro-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; LCSC C29936 -> C1525; MPN (none) -> CL05B104KO5NNNC; Manufacturer (none) -> Samsung Electro-Mechanics; Package 0603 -> 0402; now fitted; now in the parts list
- renumbered C3 to C10, C4 to C11, C5 to C12, C6 to C13, C16 to C18, C1 to C8, C2 to C9, D9 to D3, D3 to D4, D4 to D5, D5 to D6, D6 to D9, J4 to J1, J7 to J10, J13 to J11, J16 to J2, J1 to J3, J14 to J4, J5 to J6, J3 to J7, J2 to J8, J6 to J9, JP2 to JP1, R11 to R10, R9 to R11, R7 to R12, R8 to R7, R10 to R8, R12 to R9, SW3 to SW2, SW2 to SW3, U15 to U10, U4 to U11, U1 to U3, U2 to U4, U3 to U6, U14 to U9
Connections:
- net LOAD_0 is gone; now on net CLK_0: U3.14 (12_MISO_MQSL)
- net LOAD_1 is gone; now on net CLK_1: U3.22 (30_CRX3)
- net +3.3V: now also C15.2, C17.2, C2.2, C7.2, U2.8 (VCCB), U5.8 (VCCB), U7.8 (VCCB), U8.8 (VCCB); no longer C17.1
- net +5V: now also C1.2, C14.2, C16.2, C6.2, U2.1 (VCCA), U2.5 (DIR), U5.1 (VCCA), U7.1 (VCCA), U7.5 (DIR), U8.1 (VCCA); no longer C15.1
- net CLK_0: now also U5.6 (B2); no longer U3.13 (11_MOSI_CTX1)
- net CLK_1: now also U8.6 (B2); no longer U3.21 (29_TX7)
- net GND: now also C15.1, C17.1, J2.4 (Pin_4), C1.1, C14.1, C16.1, C2.1, C6.1, C7.1, U2.4 (GND), U5.4 (GND), U5.5 (DIR), U7.4 (GND), U8.4 (GND), U8.5 (DIR); no longer C15.2, C17.2, J2.12 (Pin_12)
- net SER_0: now also U2.7 (B1)
- net SER_1: now also U7.7 (B1)
- net CLK_2: no longer names the net of U3.26 (34_RX8)
- net CLK_3: no longer names the net of U3.36 (14_A0_TX3_SPDIF_OUT)
- net IO_Level_Shift/CLK_OUT renamed CLK_OUT_0
- net CLK_OUT_0: now also U5.3 (A2)
- net IO_Level_Shift/LOAD_OUT renamed LD_OUT_0
- net LD_OUT_0: now also U5.2 (A1)
- net IO_Level_Shift/SERIAL_IN renamed SER_IN_0
- net SER_IN_0: now also U2.2 (A1)
- net IO_Level_Shift1/CLK_OUT renamed CLK_OUT_1
- net CLK_OUT_1: now also U8.3 (A2)
- net IO_Level_Shift1/LOAD_OUT renamed LD_OUT_1
- net LD_OUT_1: now also U8.2 (A1)
- net IO_Level_Shift1/SERIAL_IN renamed SER_IN_1
- net SER_IN_1: now also U7.2 (A1)
- net LOAD_2: no longer names the net of U3.25 (33_MCLK2)
- net LOAD_3: no longer names the net of U3.35 (13_SCK_LED)
- net SER_2: no longer names the net of U3.27 (35_TX8)
- net SER_3: no longer names the net of U3.37 (15_A1_RX3_SPDIF_IN)
- new net LD_0: U3.13 (11_MOSI_CTX1), U5.7 (B1)
- new net LD_1: U3.21 (29_TX7), U8.7 (B1)
Other:
- removed sheet IO_Level_Shift
- removed sheet IO_Level_Shift1
- removed sheet IO_Level_Shift2
- removed sheet IO_Level_Shift3
- note added: "Level Shifting"
- moved on the sheet: C13, C18, D3, D7, F1, J1, J10, J11, J2, J4, J6, J7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
