File: Hardware/GVH_CounterController/GVH_CounterContoller.kicad_sch (KiCad schematic)
At the start: 68 parts, among them J1 Molex Micro-Fit 5pos, J10 Molex Micro-Fit 2pos, J11 Molex Micro-Fit 3pos, J2 Conn_02x08_Odd_Even, J3 Molex Ultra-Fit, J4 Molex Ultra-Fit, J6 Molex Micro-Fit 5pos, J7 WIZnet_J1B1211CCD_RJ45, J8 Molex Micro-Fit 2pos, J9 Molex Micro-Fit 2pos, K1 Relay_DPDT, Q1 MBT2222, SW2 SW_DIP_x02, SW3 SW_MEC_5G, U10 AO4882, U11 DS18B20_, U2 SN74LVC2T45, U3 Teensy4.1, U4 R-78E5.0-1.0, U5 SN74LVC2T45DCUR, U6 RT9080-3.3, U7 SN74LVC2T45DCUR, U8 SN74LVC2T45DCUR, U9 SN74LVC2G17

Commit message: Added Glass fuse and cleaned up fan controller
Parts:
- added F2: Fuse, MeowWolf_Devices:Fuseholder_2AG_5x15mm_Littelfuse_01110501Z, symbol Device:Fuse
- added JP2, JP3: SolderJumper_2_Bridged, Jumper:SolderJumper-2_P1.3mm_Bridged_RoundedPad1.0x1.5mm, symbol Jumper:SolderJumper_2_Bridged
Connections:
- net +12V: now also F2.1
- net +3.3V: now also J2.1 (Pin_1); no longer J2.2 (Pin_2)
- net +5V: now also J2.2 (Pin_2); no longer J2.1 (Pin_1)
- net FAN_CTRL_0: now also JP2.1 (A); no longer U9.1 (1A)
- net FAN_CTRL_1: now also JP3.1 (A); no longer U9.3 (2A)
- net GND: now also D1.1 (A), D1.2 (A)
- net FAN_PWR_0 renamed FAN_DRAIN_0
- net FAN_DRAIN_0: now also D8.2 (A), J10.1 (Pin_1), J9.1 (Pin_1); no longer D7.2 (A), J8.1 (Pin_1)
- removed net FAN_PWR_1: D8.2 (A), J10.1 (Pin_1), J9.1 (Pin_1), U10.5 (D), U10.6 (D)
- new net: JP2.2 (B), U9.1 (1A)
- new net: JP3.2 (B), U9.3 (2A)
- new net: F2.2, J3.2 (Pin_2)
- new net FAN_DRAIN_1: D7.2 (A), J8.1 (Pin_1), U10.5 (D), U10.6 (D)
Other:
- moved on the sheet: C18, D1, D7, J10, J8, J9, R10, R7, R8, R9, U10, U9

Commit message: About to change gate driver buffer, it wont shift logic up
Parts:
- removed D3: Reverse Protection Diode, Package_TO_SOT_SMD:TO-252-2_TabPin1, symbol Device:D
- removed F1: Fuse, MeowWolf_Devices:Fuseholder_2AG_5x15mm_Littelfuse_01110501Z, symbol Device:Fuse
- removed J2: Conn_02x08_Odd_Even, Connector_PinHeader_2.54mm:PinHeader_2x08_P2.54mm_Vertical, symbol Connector_Generic:Conn_02x08_Odd_Even
- removed J4: Molex Ultra-Fit, 0_connector:MOLEX_ULTRAFIT-RA-2POS_1723104102, symbol 0_connector:Molex Ultra-Fit 2pos IN
- added J5: Conn_02x10_Odd_Even, Connector_PinHeader_2.54mm:PinHeader_2x10_P2.54mm_Vertical, symbol Connector_Generic:Conn_02x10_Odd_Even
- renumbered D8 to D7, D7 to D8
Connections:
- net +12V: now also J5.20 (Pin_20)
- net +12V_ISO: now also J5.19 (Pin_19)
- net +3.3V: now also J5.1 (Pin_1)
- net +5V: now also J5.2 (Pin_2)
- net FAN_CTRL_0: now also U9.1 (1A)
- net FAN_CTRL_1: now also U9.3 (2A)
- net GND: now also J5.17 (Pin_17), J5.18 (Pin_18), J5.3 (Pin_3), J5.4 (Pin_4)
- net TEMP_SENS_0: now also U3.43 (21_A7_RX5_BCLK1)
- net TEMP_SENS_1: now also U3.44 (22_A8_CTX1)
- net TOUCH_RESET: now also U3.24 (32_OUT1B)
- net GPIO_11: now reaches JP2.2 (B)
- net GPIO_11: now also U3.26 (34_RX8), J5.15 (Pin_15); no longer U9.1 (1A)
- net GPIO_12: now reaches JP3.2 (B)
- net GPIO_12: now also U3.25 (33_MCLK2), J5.16 (Pin_16); no longer U9.3 (2A)
- net GPIO_10: now reaches U3.27 (35_TX8)
- net GPIO_10: now also J5.14 (Pin_14)
- net GPIO_9: now reaches U3.28 (36_CS)
- net GPIO_9: now also J5.13 (Pin_13)
- net GPIO_8: now reaches U3.29 (37_CS)
- net GPIO_8: now also J5.12 (Pin_12)
- net GPIO_7: now reaches U3.30 (38_CS1_IN1)
- net GPIO_7: now also J5.11 (Pin_11)
- net GPIO_6: now reaches U3.31 (39_MISO1_OUT1A)
- net GPIO_6: now also J5.10 (Pin_10)
- net GPIO_5: now reaches U3.32 (40_A16)
- net GPIO_5: now also J5.9 (Pin_9)
- net GPIO_4: now reaches U3.33 (41_A17)
- net GPIO_4: now also J5.8 (Pin_8)
- net GPIO_3: now reaches U3.38 (16_A2_RX4_SCL1)
- net GPIO_3: now also J5.7 (Pin_7)
- net GPIO_2: now reaches U3.39 (17_A3_TX4_SDA1)
- net GPIO_2: now also J5.6 (Pin_6)
- net GPIO_1: now reaches U3.40 (18_A4_SDA)
- net GPIO_1: now also J5.5 (Pin_5)

Commit message: Controller board finished and documentation created
Parts:
- removed C18: 0.1uF, Capacitor_SMD:C_0402_1005Metric, symbol Device:C_Small
- removed U9: SN74LVC2G17, Package_TO_SOT_SMD:SOT-23-6, symbol 0_integrated_circuits:SN74LVC2G17
- added C13, C14: 0.1uF, Capacitor_SMD:C_0402_1005Metric, symbol Device:C_Small
- added R1, R13, R14, R2: 68R, Resistor_SMD:R_0402_1005Metric, symbol Device:R_Small
- added U7: SN74LVC2T45DCUR, Package_SO:VSSOP-8_2.4x2.1mm_P0.5mm, symbol Logic_LevelTranslator:SN74LVC2T45DCUR
- C1, C2, C6, C7: Digikey Page https://www.digikey.com/en/products/detail/samsung-electro-mechanics/CL05B104KO5NNNC/3886659?s=N4IgTCBcDaIMIBkAMBWAQgRiQFgNIHkUA5EuEAXQF8g -> https://www.digikey.com/en/products/detail/samsung-electro-mechanics/CL05B104KO5NNNC/3886659; MPN CL05B104KO5NNNC -> (none); Manu # (none) -> CL05B104KO5NNNC; Manu. (none) -> Samsung Electro-Mechanics; Manufacturer Samsung Electro-Mechanics -> (none)
- C10: renamed from C12; MPN CL21A106KAYNNNE -> (none); Manu # (none) -> CL21A106KAYNNNE; Manu. (none) -> Samsung Electro-Mechanics; Manufacturer Samsung Electro-Mechanics -> (none)
- C11: renamed from C14; Digikey Page https://www.digikey.com/en/products/detail/samsung-electro-mechanics/CL05B104KO5NNNC/3886659?s=N4IgTCBcDaIMIBkAMBWAQgRiQFgNIHkUA5EuEAXQF8g -> https://www.digikey.com/en/products/detail/samsung-electro-mechanics/CL05B104KO5NNNC/3886659; MPN CL05B104KO5NNNC -> (none); Manu # (none) -> CL05B104KO5NNNC; Manu. (none) -> Samsung Electro-Mechanics; Manufacturer Samsung Electro-Mechanics -> (none)
- C12: renamed from C15; Digikey Page https://www.digikey.com/en/products/detail/samsung-electro-mechanics/CL05B104KO5NNNC/3886659?s=N4IgTCBcDaIMIBkAMBWAQgRiQFgNIHkUA5EuEAXQF8g -> https://www.digikey.com/en/products/detail/samsung-electro-mechanics/CL05B104KO5NNNC/3886659; MPN CL05B104KO5NNNC -> (none); Manu # (none) -> CL05B104KO5NNNC; Manu. (none) -> Samsung Electro-Mechanics; Manufacturer Samsung Electro-Mechanics -> (none)
- C15: renamed from C16; Digikey Page https://www.digikey.com/en/products/detail/samsung-electro-mechanics/CL05B104KO5NNNC/3886659?s=N4IgTCBcDaIMIBkAMBWAQgRiQFgNIHkUA5EuEAXQF8g -> https://www.digikey.com/en/products/detail/samsung-electro-mechanics/CL05B104KO5NNNC/3886659; MPN CL05B104KO5NNNC -> (none); Manu # (none) -> CL05B104KO5NNNC; Manu. (none) -> Samsung Electro-Mechanics; Manufacturer Samsung Electro-Mechanics -> (none)
- C16: renamed from C17; Digikey Page https://www.digikey.com/en/products/detail/samsung-electro-mechanics/CL05B104KO5NNNC/3886659?s=N4IgTCBcDaIMIBkAMBWAQgRiQFgNIHkUA5EuEAXQF8g -> https://www.digikey.com/en/products/detail/samsung-electro-mechanics/CL05B104KO5NNNC/3886659; MPN CL05B104KO5NNNC -> (none); Manu # (none) -> CL05B104KO5NNNC; Manu. (none) -> Samsung Electro-Mechanics; Manufacturer Samsung Electro-Mechanics -> (none)
- C3: renamed from C8; Digikey Page https://www.digikey.com/en/products/detail/samsung-electro-mechanics/CL31B106KBHNNNE/5961251?s=N4IgTCBcDaIMIBkDMBGAQigDANgNJoAkA5EgURAF0BfIA -> https://www.digikey.com/en/products/detail/samsung-electro-mechanics/CL31B106KBHNNNE/5961251; MPN CL31B106KBHNNNE -> (none); Manu # (none) -> CL31B106KBHNNNE; Manu. (none) -> Samsung Electro-Mechanics; Manufacturer Samsung Electro-Mechanics -> (none)
- C4: renamed from C9; Digikey Page https://www.digikey.com/en/products/detail/samsung-electro-mechanics/CL31B106KBHNNNE/5961251?s=N4IgTCBcDaIMIBkDMBGAQigDANgNJoAkA5EgURAF0BfIA -> https://www.digikey.com/en/products/detail/samsung-electro-mechanics/CL31B106KBHNNNE/5961251; MPN CL31B106KBHNNNE -> (none); Manu # (none) -> CL31B106KBHNNNE; Manu. (none) -> Samsung Electro-Mechanics; Manufacturer Samsung Electro-Mechanics -> (none)
- C5: renamed from C10; Digikey Page https://www.digikey.com/en/products/detail/samsung-electro-mechanics/CL31B106KBHNNNE/5961251?s=N4IgTCBcDaIMIBkDMBGAQigDANgNJoAkA5EgURAF0BfIA -> https://www.digikey.com/en/products/detail/samsung-electro-mechanics/CL31B106KBHNNNE/5961251; MPN CL31B106KBHNNNE -> (none); Manu # (none) -> CL31B106KBHNNNE; Manu. (none) -> Samsung Electro-Mechanics; Manufacturer Samsung Electro-Mechanics -> (none)
- C8: renamed from C13; Digikey Page https://www.digikey.com/en/products/detail/samsung-electro-mechanics/CL21B104KBCNNNC/3886661?s=N4IgTCBcDaIMIBkwEYBCyAMAWA0quAckXCALoC%2BQA -> https://www.digikey.com/en/products/detail/samsung-electro-mechanics/CL21B104KBCNNNC/3886661; MPN CL21B104KBCNNNC -> (none); Manu # (none) -> CL21B104KBCNNNC; Manu. (none) -> Samsung Electro-Mechanics; Manufacturer Samsung Electro-Mechanics -> (none)
- C9: renamed from C11; MPN CL21A106KAYNNNE -> (none); Manu # (none) -> CL21A106KAYNNNE; Manu. (none) -> Samsung Electro-Mechanics; Manufacturer Samsung Electro-Mechanics -> (none)
- D1: Digikey P/N (none) -> 1727-1904-1-ND; Digikey Page (none) -> https://www.digikey.com/en/products/detail/nexperia-usa-inc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; Manu # (none) -> PMEG045V100EPDZ; Manu. (none) -> Nexperia USA Inc.; Package TO-277 -> CFP-15
- D2: Digikey P/N - -> LTST-C190KRKT; Digikey Page - -> https://www.digikey.com/en/products/detail/liteon/LTST-C190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; MPN LTST-C190KRKT -> (none); Manu # (none) -> LTST-C190KRKT; Manu. (none) -> Lite-On; Manufacturer Lite-On -> (none)
- D3: renamed from D4; Digikey P/N - -> 1N4148WS-FDICT-ND; Digikey Page - -> https://www.digikey.com/en/products/detail/diodes-incorpora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; MPN 1N4148WS -> (none); Manu # (none) -> 1N4148WS; Manu. (none) -> Jiangsu Changjing Electronics Technology Co., Ltd.; Manufacturer Jiangsu Changjing Electronics Technology Co., Ltd. -> (none)
- D4: renamed from D5; Digikey P/N - -> 160-1888-1-ND; Digikey Page - -> https://www.digikey.com/en/products/detail/liteon/LTST-C191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; MPN LTST-C191TGKT -> (none); Manu # (none) -> LTST-C191TGKT; Manu. (none) -> Lite-On; Manufacturer Lite-On -> (none)
- D5: renamed from D6; Digikey P/N - -> LTST-C190KRKT; Digikey Page - -> https://www.digikey.com/en/products/detail/liteon/LTST-C190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; MPN LTST-C190KRKT -> (none); Manu # (none) -> LTST-C190KRKT; Manu. (none) -> Lite-On; Manufacturer Lite-On -> (none)
- D6: renamed from D7; MPN PMEG10030ELPX -> (none); Manu # (none) -> PMEG10030ELPX; Manu. (none) -> Nexperia USA Inc.; Manufacturer Nexperia -> (none)
- D7: renamed from D8; MPN PMEG10030ELPX -> (none); Manu # (none) -> PMEG10030ELPX; Manu. (none) -> Nexperia USA Inc.; Manufacturer Nexperia -> (none)
- D8: renamed from D9; Digikey P/N - -> 1528-4684-ND; Digikey Page - -> https://www.digikey.com/en/products/detail/adafruit-industr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; MPN WS2812B-2020 -> (none); Manu # (none) -> WS2812B-2020; Manu. (none) -> Worldsemi; Manufacturer Worldsemi -> (none)
- F1: renamed from F2; Digikey Page https://www.digikey.com/en/products/detail/littelfuse-inc/01110501Z/2518598?s=N4IgTCBcDaIDIEsAuSCmAbAZgVwM6oAIAGARjKIFZSAtEAXQF8g -> https://www.digikey.com/en/products/detail/littelfuse-inc/01110501Z/2518598; MPN 01110501Z -> (none); Manu # (none) -> 01110501Z; Manu. (none) -> Littelfuse Inc.; Manufacturer Littelfuse Inc. -> (none)
- H1, H2, H3, H4: MPN - -> (none); Manu. (none) -> -; Manufacturer - -> (none)
- J1: renamed from J3; Digikey Page https://www.digikey.com/en/products/detail/molex/1723104102/14122202?s=N4IgTCBcDaIIwHYwGY4AYC0AWdEC6AvkA -> https://www.digikey.com/en/products/detail/molex/1723104102/14122202; MPN 1723104102 -> (none); Manu # (none) -> 1723104102; Manu. (none) -> MOLEX; Manufacturer MOLEX -> (none)
- J2: renamed from J5; value Conn_02x10_Odd_Even -> Vertical Header Pins; Digikey P/N (none) -> 2057-PH2-20-UA-ND; Digikey Page (none) -> https://www.digikey.com/en/products/detail/adam-tech/PH2-20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; LCSC (none) -> -; Manu # (none) -> PH2-20-UA; Manu. (none) -> Adam Tech; Package (none) -> THT
- J3: renamed from J7; LCSC (none) -> -; Manu # (none) -> J1B1211CCD; Manu. (none) -> WIZnet; Manufacturer WIZnet -> (none); Mfg. P/N J1B1211CCD -> (none); Package (none) -> THT
- J4: renamed from J9; value Molex Micro-Fit 2pos -> Molex Micro-Fit; LCSC (none) -> -; Manu # (none) -> 0436500215; Manu. (none) -> MOLEX; Manufacturer MOLEX -> (none); Mfg. P/N 0436500215 -> (none); Package (none) -> THT
- J5: renamed from J1; value Molex Micro-Fit 5pos -> Molex Micro-Fit; Digikey Page https://www.digikey.com/en/products/detail/molex/0436500500/268992?s=N4IgTCBcDaIAwBYDMA2ArHOG4gLoF8g -> https://www.digikey.com/en/products/detail/molex/0436500500/268992; LCSC (none) -> -; MPN 0436500500 -> (none); Manu # (none) -> 0436500500; Manu. (none) -> MOLEX; Manufacturer MOLEX -> (none); Package (none) -> THT
- J6: renamed from J10; value Molex Micro-Fit 2pos -> Molex Micro-Fit; LCSC (none) -> -; Manu # (none) -> 0436500215; Manu. (none) -> MOLEX; Manufacturer MOLEX -> (none); Mfg. P/N 0436500215 -> (none); Package (none) -> THT
- J7: renamed from J8; value Molex Micro-Fit 2pos -> Molex Micro-Fit; LCSC (none) -> -; Manu # (none) -> 0436500215; Manu. (none) -> MOLEX; Manufacturer MOLEX -> (none); Mfg. P/N 0436500215 -> (none); Package (none) -> THT
- J8: renamed from J6; value Molex Micro-Fit 5pos -> Molex Micro-Fit; Digikey Page https://www.digikey.com/en/products/detail/molex/0436500500/268992?s=N4IgTCBcDaIAwBYDMA2ArHOG4gLoF8g -> https://www.digikey.com/en/products/detail/molex/0436500500/268992; LCSC (none) -> -; MPN 0436500500 -> (none); Manu # (none) -> 0436500500; Manu. (none) -> MOLEX; Manufacturer MOLEX -> (none); Package (none) -> THT
- J9: renamed from J11; value Molex Micro-Fit 3pos -> Molex Micro-Fit; LCSC (none) -> -; Manu # (none) -> 0436500315; Manu. (none) -> MOLEX; Manufacturer MOLEX -> (none); Mfg. P/N 0436500315 -> (none); Package (none) -> THT
- K1: LCSC (none) -> -; MPN EC2-3NU -> (none); Manu # (none) -> EC2-3NU; Manu. (none) -> KEMET; Manufacturer KEMET -> (none); Package (none) -> THT
- L1: Digikey P/N - -> 535-ASPI-4030S-120M-TCT-ND; Digikey Page - -> https://www.digikey.com/en/products/detail/abracon-llc/ASPI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; MPN FNR4030S120MT -> (none); Manu # (none) -> FNR4030S120MT; Manu. (none) -> Changjiang Microelectronics Tech; Manufacturer Changjiang Microelectronics Tech -> (none)
- LOGO1: MPN - -> (none); Manu # (none) -> -; Manu. (none) -> -; Manufacturer - -> (none)
- Q1: Digikey P/N - -> MMBT2222ALT1GOSCT-ND; Digikey Page - -> https://www.digikey.com/en/products/detail/onsemi/MMBT2222A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; MPN MMBT2222ALT1G -> (none); Manu # (none) -> MMBT2222ALT1G; Manu. (none) -> onsemi; Manufacturer onsemi -> (none)
- R10: renamed from R8; Digikey P/N - -> 311-100HRCT-ND; Digikey Page - -> https://www.digikey.com/en/products/detail/yageo/RC0603FR-0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; MPN RC0603FR-071KL -> (none); Manu # (none) -> RC0603FR-07100RL; Manu. (none) -> YAGEO; Manufacturer YAGEO -> (none)
- R11: renamed from R9; Digikey P/N (none) -> 311-10.0KHRCT-ND; Digikey Page (none) -> https://www.digikey.com/en/products/detail/yageo/RC0603FR-0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; Manu # (none) -> RC0603FR-0710KL; Manu. (none) -> YAGEO
- R12: renamed from R10; Digikey P/N (none) -> 311-10.0KHRCT-ND; Digikey Page (none) -> https://www.digikey.com/en/products/detail/yageo/RC0603FR-0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; Manu # (none) -> RC0603FR-0710KL; Manu. (none) -> YAGEO
- R15: renamed from R11; Digikey P/N - -> 311-4.70KHRCT-ND; Digikey Page - -> https://www.digikey.com/en/products/detail/yageo/RC0603FR-0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; MPN RC0603FR-074K7L -> (none); Manu # (none) -> RC0603FR-074K7L; Manu. (none) -> YAGEO; Manufacturer YAGEO -> (none)
- R16: renamed from R12; Digikey P/N - -> 311-4.70KHRCT-ND; Digikey Page - -> https://www.digikey.com/en/products/detail/yageo/RC0603FR-0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; MPN RC0603FR-074K7L -> (none); Manu # (none) -> RC0603FR-074K7L; Manu. (none) -> YAGEO; Manufacturer YAGEO -> (none)
- R3: renamed from R1; Digikey P/N - -> 311-1.00KHRCT-ND; Digikey Page - -> https://www.digikey.com/en/products/detail/yageo/RC0603FR-0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; MPN RC0603FR-071KL -> (none); Manu # (none) -> RC0603FR-071KL; Manu. (none) -> YAGEO; Manufacturer YAGEO -> (none)
- R4: Digikey P/N (none) -> 311-10.0KHRCT-ND; Digikey Page (none) -> https://www.digikey.com/en/products/detail/yageo/RC0603FR-0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; Manu # (none) -> RC0603FR-0710KL; Manu. (none) -> YAGEO
- R5: renamed from R2; Digikey P/N - -> 311-1.00KHRCT-ND; Digikey Page - -> https://www.digikey.com/en/products/detail/yageo/RC0603FR-0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; MPN RC0603FR-071KL -> (none); Manu # (none) -> RC0603FR-071KL; Manu. (none) -> YAGEO; Manufacturer YAGEO -> (none)
- R6: renamed from R3; Digikey P/N (none) -> 311-10.0KHRCT-ND; Digikey Page (none) -> https://www.digikey.com/en/products/detail/yageo/RC0603FR-0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; Manu # (none) -> RC0603FR-0710KL; Manu. (none) -> YAGEO
- R7: renamed from R5; Digikey P/N - -> 311-1.00KHRCT-ND; Digikey Page - -> https://www.digikey.com/en/products/detail/yageo/RC0603FR-0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; MPN RC0603FR-071KL -> (none); Manu # (none) -> RC0603FR-071KL; Manu. (none) -> YAGEO; Manufacturer YAGEO -> (none)
- R8: renamed from R6; Digikey P/N - -> 311-1.00KHRCT-ND; Digikey Page - -> https://www.digikey.com/en/products/detail/yageo/RC0603FR-0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; MPN RC0603FR-071KL -> (none); Manu # (none) -> RC0603FR-071KL; Manu. (none) -> YAGEO; Manufacturer YAGEO -> (none)
- R9: renamed from R7; Digikey P/N - -> 311-100HRCT-ND; Digikey Page - -> https://www.digikey.com/en/products/detail/yageo/RC0603FR-0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; MPN RC0603FR-071KL -> (none); Manu # (none) -> RC0603FR-07100RL; Manu. (none) -> YAGEO; Manufacturer YAGEO -> (none)
- SW1: renamed from SW2; MPN CHS-02TB -> (none); Manu # (none) -> CHS-02TB; Manu. (none) -> Nidec Components Corporation; Manufacturer Nidec Components Corporation -> (none)
- SW2: renamed from SW3; MPN B3F-1020 -> (none); Manu # (none) -> B3F-1020; Manu. (none) -> Omron Electronics Inc-EMC Div; Manufacturer Omron Electronics Inc-EMC Div -> (none)
- U1: renamed from U3; Digikey P/N (none) -> 1568-DEV-16996-ND; Digikey Page (none) -> https://www.digikey.com/en/products/detail/sparkfun-electro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; Manu # (none) -> Teensy4.1; Manu. (none) -> PJRC; Package (none) -> THT
- U10: renamed from U11; MPN DS18B20+ -> (none); Manu # (none) -> DS18B20+; Manu. (none) -> Maxim Integrated; Manufacturer Maxim Integrated -> (none)
- U2: value SN74LVC2T45 -> SN74LVC2T45DCUR; MPN SN74LVC2T45DCUT -> (none); Manu # (none) -> SN74LVC2T45DCUT; Manu. (none) -> Texas Instruments; Manufacturer Texas Instruments -> (none)
- U3: renamed from U4; MPN R-78E5.0-1.0 -> (none); Manu # (none) -> R-78E5.0-1.0; Manu. (none) -> RECOM Power; Manufacturer RECOM Power -> (none)
- U4: renamed from U5; MPN SN74LVC2T45DCUT -> (none); Manu # (none) -> SN74LVC2T45DCUT; Manu. (none) -> Texas Instruments; Manufacturer Texas Instruments -> (none)
- U5: renamed from U6; Digikey P/N (none) -> 1028-1509-1-ND; Digikey Page (none) -> https://www.digikey.com/en/products/detail/richtek-usa-inc/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; Manu # (none) -> RT9080-33GJ5; Manu. (none) -> Richtek USA Inc.
- U6: renamed from U7; MPN SN74LVC2T45DCUT -> (none); Manu # (none) -> SN74LVC2T45DCUT; Manu. (none) -> Texas Instruments; Manufacturer Texas Instruments -> (none)
- U8: renamed from U10; Manu # (none) -> AO4882; Manu. (none) -> Alpha & Omega Semiconductor; Manufacturer Alpha & Omega Semiconductor -> (none); Mfg. P/N AO4882 -> (none)
- U9: renamed from U8; MPN SN74LVC2T45DCUT -> (none); Manu # (none) -> SN74LVC2T45DCUT; Manu. (none) -> Texas Instruments; Manufacturer Texas Instruments -> (none)
- renumbered JP2 to JP1, JP3 to JP2, JP1 to JP3
Connections:
- net +3.3V: now also C13.2, U7.1 (VCCA), U7.5 (DIR)
- net +5V: now also C14.2, U7.8 (VCCB)
- net CLK_OUT_0: now also R2.1; no longer U4.3 (A2)
- net CLK_OUT_1: now also R14.1; no longer U9.3 (A2)
- net FAN_CTRL_0: now also U7.2 (A1)
- net FAN_CTRL_1: now also U7.3 (A2)
- net GND: now also C13.1, C14.1, U7.4 (GND)
- net LD_OUT_0: now also R1.1; no longer U4.2 (A1)
- net LD_OUT_1: now also R13.1; no longer U9.2 (A1)
- net at R10.1, R12.2: now also U7.6 (B2)
- net at R11.2, R9.1: now also U7.7 (B1)
- new net: R1.2, U4.2 (A1)
- new net: R14.2, U9.3 (A2)
- new net: R2.2, U4.3 (A2)
- new net: R13.2, U9.2 (A1)
Other:
- note added: "20 Pin GPIO"
- note added: "Fan Connectors"
- note added: "Teensy With Ethernet"
- note added: "Touch Board Connectors"
- title: (none) -> Interactive Counter Controller
- moved on the sheet: C1, C10, C11, C12, C15, C16, C2, C3, C4, C5, C6, C7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
